File: FYP-METRO-SHIELD.kicad_pcb (KiCad board)
At the start: 2 copper layers, 68.6 x 53.3 mm, 8 parts, among them J1 Power, J2 Digital/PWM, J3 Analog, J4 Digital/PWM

Commit message: aaa
Parts:
- added C1: 0.1u, Capacitor_SMD:C_0805_2012Metric, F.Cu at (122.0, 85.0)
- added C10: 100n, Capacitor_SMD:C_0805_2012Metric, F.Cu at (53.0, 38.1)
- added C2: 0.1u, Capacitor_SMD:C_0805_2012Metric, F.Cu at (132.0, 89.0)
- added C3: 100n, Capacitor_SMD:C_0805_2012Metric, F.Cu at (149.9, 85.5)
- added C4: 100n, Capacitor_SMD:C_0805_2012Metric, F.Cu at (191.0, 26.9)
- added C5: 100n, Capacitor_SMD:C_0805_2012Metric, F.Cu at (191.0, 30.0)
- added C6: 47n, Capacitor_SMD:C_0805_2012Metric, F.Cu at (191.0, 33.0)
- added C7: 100n, Capacitor_SMD:C_0805_2012Metric, F.Cu at (191.0, 36.0)
- added C8: 100n, Capacitor_SMD:C_0805_2012Metric, F.Cu at (41.0, 36.2)
- added C9: 100n, Capacitor_SMD:C_0805_2012Metric, F.Cu at (31.7, 35.0)
- added D1: BZT52C2V0-7-F, Diode_SMD:D_SOD-123F, F.Cu at (158.3, 86.5)
- added D2: D_Schottky, Diode_SMD:D_SOD-123, F.Cu at (183.2, 40.3)
- added D3: D_Schottky, Diode_SMD:D_SOD-123, F.Cu at (40.8, 30.6)
- added D4: D_Schottky, Diode_SMD:D_SOD-123, F.Cu at (85.3, 35.0)
- added J5: Conn_01x02_Socket, Connector_PinHeader_2.54mm:PinHeader_1x02_P2.54mm_Vertical, F.Cu at (209.9, 44.0)
- added J6: Conn_01x02_Socket, Connector_PinHeader_2.54mm:PinHeader_1x02_P2.54mm_Vertical, F.Cu at (53.4, 67.3)
- added J7: Conn_01x04_Socket, Connector_PinHeader_2.54mm:PinHeader_1x04_P2.54mm_Vertical, F.Cu at (137.8, 84.0)
- added JP1: Jumper_3_Bridged12, Jumper:SolderJumper-3_P1.3mm_Bridged12_RoundedPad1.0x1.5mm_NumberLabels, F.Cu at (119.5, 82.5)
- added JP2: Jumper_3_Bridged12, Jumper:SolderJumper-3_P1.3mm_Bridged12_RoundedPad1.0x1.5mm_NumberLabels, F.Cu at (80.8, 47.4)
- added Q1: BC847, Package_TO_SOT_SMD:SOT-23, F.Cu at (127.0, 90.0)
- added R1: 10k, Resistor_SMD:R_0805_2012Metric, F.Cu at (122.0, 87.0)
- added R10: 1M, Resistor_SMD:R_0805_2012Metric, F.Cu at (141.7, 87.0)
- added R11: 1M, Resistor_SMD:R_0805_2012Metric, F.Cu at (141.7, 93.1)
- added R12: 1.4k, Resistor_SMD:R_0805_2012Metric, F.Cu at (195.4, 26.9)
- added R13: 1.4k, Resistor_SMD:R_0805_2012Metric, F.Cu at (195.4, 29.9)
- added R14: 10k, Resistor_SMD:R_0805_2012Metric, F.Cu at (195.4, 32.8)
- added R15: 10k, Resistor_SMD:R_0805_2012Metric, F.Cu at (31.7, 39.0)
- added R16: 300k, Resistor_SMD:R_0805_2012Metric, F.Cu at (31.7, 37.0)
- added R17: 10k, Resistor_SMD:R_0805_2012Metric, F.Cu at (31.7, 33.0)
- added R18: 10k, Resistor_SMD:R_0805_2012Metric, F.Cu at (48.6, 56.3)
- added R19: 300k, Resistor_SMD:R_0805_2012Metric, F.Cu at (52.5, 43.0)
- added R2: 370k, Resistor_SMD:R_0805_2012Metric, F.Cu at (122.0, 89.0)
- added R20: 3.3k, Resistor_SMD:R_0805_2012Metric, F.Cu at (69.6, 46.2)
- added R21: 10k, Resistor_SMD:R_0805_2012Metric, F.Cu at (69.6, 49.1)
- added R3: 1.4k, Resistor_SMD:R_0805_2012Metric, F.Cu at (122.0, 91.0)
- added R4: 10k, Resistor_SMD:R_0805_2012Metric, F.Cu at (132.0, 91.0)
- added R5: 1k, Resistor_SMD:R_0805_2012Metric, F.Cu at (158.3, 89.0)
- added R6: 10k, Resistor_SMD:R_0805_2012Metric, F.Cu at (141.7, 88.9)
- added R7: 10k, Resistor_SMD:R_0805_2012Metric, F.Cu at (141.7, 91.1)
- added R8: 9.1k, Resistor_SMD:R_0805_2012Metric, F.Cu at (158.3, 93.0)
- added R9: 1k, Resistor_SMD:R_0805_2012Metric, F.Cu at (158.3, 91.0)
- added RV1: 10k, Potentiometer_SMD:Potentiometer_Bourns_TC33X_Vertical, F.Cu at (122.0, 94.2)
- added RV2: 10k, Potentiometer_SMD:Potentiometer_Bourns_TC33X_Vertical, F.Cu at (191.9, 39.9)
- added RV3: 10k, Potentiometer_SMD:Potentiometer_Bourns_TC33X_Vertical, F.Cu at (31.7, 42.0)
- added RV4: 10k, Potentiometer_SMD:Potentiometer_Bourns_TC33X_Vertical, F.Cu at (49.3, 48.8)
- added RV5: 10k, Potentiometer_SMD:Potentiometer_Bourns_TC33X_Vertical, F.Cu at (75.0, 41.9)
- added U1: MCP602, Package_SO:SOIC-8_3.9x4.9mm_P1.27mm, F.Cu at (150.0, 90.0)
- added U2: LM386, Package_SO:SOIC-8_3.9x4.9mm_P1.27mm, F.Cu at (184.5, 28.8)
- added U3: LM393, Package_SO:SOIC-8_3.9x4.9mm_P1.27mm, F.Cu at (184.5, 35.4)
- added U4: MCP602, Package_SO:SOIC-8_3.9x4.9mm_P1.27mm, F.Cu at (40.0, 40.0)
Connections:
- J3 pad 3: /A2 -> 0.5V
Routing:
- net 0.5V: track 0.00 -> 23.3 mm, vias 0 -> 1
- net Net-(D1-K): track 0.00 -> 20.8 mm
- net /A1: track 0.00 -> 20.0 mm, vias 0 -> 1
- net /A0: track 0.00 -> 18.6 mm
- net +5V: track 0.00 -> 13.6 mm
- net /IR Sensor/PT_in: track 0.00 -> 13.4 mm
- net Net-(JP1-C): track 0.00 -> 13.1 mm
- net Net-(Q1-C): track 0.00 -> 11.6 mm
- net /Magnet Sensor/MAG_in: track 0.00 -> 9.88 mm
- net Net-(Q1-B): track 0.00 -> 8.07 mm
- net Net-(U1A-+): track 0.00 -> 7.86 mm
- net Net-(U1A--): track 0.00 -> 7.81 mm
- net Net-(U1B-+): track 0.00 -> 6.91 mm
- net +3V3: track 0.00 -> 4.08 mm
- net /A3: track 0.00 -> 2.02 mm
