File: FYP-METRO-SHIELD.kicad_pcb (KiCad board)
At the start: 2 copper layers, 68.6 x 53.3 mm, 58 parts, among them J1 Power, J2 Digital/PWM, J3 Analog, J4 Digital/PWM, J5 Conn_01x02_Socket, J6 Conn_01x02_Socket, J7 Conn_01x04_Socket, Q1 BC847, U1 MCP602, U2 LM386, U3 LM393, U4 MCP602

Commit message: Add files via upload
Parts:
- removed JP1, JP2: Jumper_3_Bridged12, Jumper:SolderJumper-3_P1.3mm_Bridged12_RoundedPad1.0x1.5mm_NumberLabels
- removed RV1, RV3, RV4: 10k, Potentiometer_SMD:Potentiometer_Bourns_TC33X_Vertical
- added D5: LED, LED_THT:LED_D3.0mm, F.Cu at (116.0, 92.3)
- added J10: Conn_01x03_Socket, Connector_PinHeader_2.54mm:PinHeader_1x03_P2.54mm_Vertical, F.Cu at (166.0, 81.5)
- added J8: Conn_01x03_Pin, Connector_PinHeader_2.54mm:PinHeader_1x03_P2.54mm_Vertical, F.Cu at (119.0, 85.9)
- added J9: Conn_01x03_Pin, Connector_PinHeader_2.54mm:PinHeader_1x03_P2.54mm_Vertical, F.Cu at (127.5, 71.0)
- added R22: 3.3k, Resistor_THT:R_Axial_DIN0204_L3.6mm_D1.6mm_P5.08mm_Horizontal, F.Cu at (114.3, 80.1)
- C1, C2: value 0.1u -> 100n; footprint Capacitor_SMD:C_0805_2012Metric -> Capacitor_THT:C_Disc_D3.0mm_W2.0mm_P2.50mm
- C10, C3, C4, C5, C6, C7, C8, C9: footprint Capacitor_SMD:C_0805_2012Metric -> Capacitor_THT:C_Disc_D3.0mm_W2.0mm_P2.50mm
- D1: footprint Diode_SMD:D_SOD-123F -> Resistor_THT:R_Axial_DIN0204_L3.6mm_D1.6mm_P5.08mm_Horizontal
- D2, D4: value D_Schottky -> ~; footprint Diode_SMD:D_SOD-123 -> Diode_THT:D_DO-34_SOD68_P7.62mm_Horizontal
- D3: footprint Diode_SMD:D_SOD-123 -> Diode_THT:D_DO-34_SOD68_P7.62mm_Horizontal
- J7: value Conn_01x04_Socket -> Conn_01x02_Socket; footprint Connector_PinHeader_2.54mm:PinHeader_1x04_P2.54mm_Vertical -> Connector_PinHeader_2.54mm:PinHeader_1x02_P2.54mm_Vertical
- Q1: value BC847 -> BC547; footprint Package_TO_SOT_SMD:SOT-23 -> Package_TO_SOT_THT:TO-92_Inline
- R1, R10, R11, R12, R13, R14, R15, R16, R17, R18, R19, R20, R21, R3, R4, R5, R6, R7, R8, R9: footprint Resistor_SMD:R_0805_2012Metric -> Resistor_THT:R_Axial_DIN0204_L3.6mm_D1.6mm_P5.08mm_Horizontal
- R2: value 370k -> 390k; footprint Resistor_SMD:R_0805_2012Metric -> Resistor_THT:R_Axial_DIN0204_L3.6mm_D1.6mm_P5.08mm_Horizontal
- RV2, RV5: footprint Potentiometer_SMD:Potentiometer_Bourns_TC33X_Vertical -> Potentiometer_THT:Potentiometer_Bourns_3386F_Vertical
- U1, U2, U3, U4: footprint Package_SO:SOIC-8_3.9x4.9mm_P1.27mm -> Package_DIP:DIP-8_W7.62mm_Socket
- moved R17 96.1 mm to (120.0, 71.0), turned to -90 degrees
- moved C9 93.3 mm to (119.2, 67.5)
- moved D3 91.6 mm to (123.0, 71.0), turned to -90 degrees
- moved C8 84.5 mm to (123.8, 53.0)
- moved R15 84.3 mm to (113.0, 61.5), turned to -90 degrees
- moved R16 82.9 mm to (113.0, 53.5), turned to -90 degrees
- moved C10 81.8 mm to (133.0, 55.2), turned to -90 degrees
- moved R18 78.7 mm to (127.0, 62.5), turned to -90 degrees
- moved U4 77.9 mm to (116.2, 56.2)
- moved R19 75.5 mm to (127.0, 55.0), turned to -90 degrees
- moved R21 73.1 mm to (138.5, 73.5), turned to 90 degrees
- moved C5 68.6 mm to (136.0, 71.0), turned to 90 degrees
- moved RV5 68.1 mm to (134.2, 75.5), turned to 180 degrees
- moved R14 67.6 mm to (141.5, 73.5), turned to 90 degrees
- moved R20 65.0 mm to (133.0, 60.5), turned to -90 degrees
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Connections:
- J2 pad 1: /SCL/A5 -> unconnected-(J2-Pin_1-Pad1)
- J2 pad 2: /SDA/A4 -> unconnected-(J2-Pin_2-Pad2)
- J7 pad 1: +5V -> /IR Sensor/PT_in
- J7 pad 2: /Magnet Sensor/MAG_in -> GND
- Q1 pad 1: Net-(Q1-B) -> Net-(Q1-C)
- Q1 pad 2: GND -> Net-(Q1-B)
- Q1 pad 3: Net-(Q1-C) -> GND
Routing:
- net +5V: track 13.6 -> 164.0 mm
- net +3V3: track 4.08 -> 102.5 mm
- net /A3: track 2.02 -> 50.2 mm
- net 0.5V: track 23.3 -> 53.2 mm, vias 1 -> 0
- net /7: track 0.00 -> 23.3 mm
- net /8: track 0.00 -> 22.9 mm
- net Net-(D4-K): track 0.00 -> 19.6 mm
- net Net-(D2-K): track 0.00 -> 18.2 mm
- net Net-(C9-Pad1): track 0.00 -> 17.9 mm
- net Net-(D1-K): track 20.8 -> 4.60 mm
- net Net-(J9-Pin_2): track 0.00 -> 15.9 mm
- net /A1: track 20.0 -> 33.7 mm, vias 1 -> 0
- net /Magnet Sensor/MAG_in: track 9.88 -> 23.5 mm
- net Net-(U2-+): track 0.00 -> 12.7 mm
- net Net-(U3A--): track 0.00 -> 12.3 mm
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- added copper zone on B.Cu, net GND
- added copper zone on F.Cu, net GND
Other:
- board size 68.6 x 53.3 mm -> 57.1 x 53.3 mm
- board text added: "3V3"
- board text added: "5V"
- board text removed: "ICSP"
