File: SENSOR_RADIO.kicad_sch (KiCad schematic)
At the start: 0 parts

Commit message: LOL
Parts:
- added C10, C8, C9: 100n, Capacitor_SMD:C_0805_2012Metric, symbol Device:C
- added D4: D, symbol Device:D
- added R15, R19: 300k, Resistor_SMD:R_0805_2012Metric, symbol Device:R
- added R16, R17, R18: 10k, Resistor_SMD:R_0805_2012Metric, symbol Device:R
- added R20: 3.3k, Resistor_SMD:R_0805_2012Metric, symbol Device:R
- added U4: MCP602, symbol Amplifier_Operational:MCP602
Connections:
- new net: C9.1, R15.1, U4.1
- new net: R15.2, R16.1, U4.2 (-)
- new net: C9.2, R17.1, R18.2
- new net: R18.1, R19.2, U4.6 (-)
- new net: D4.2 (A), U4.7
- new net: C10.2, D4.1 (K), R19.1, R20.1
- new net +3V3: U4.3 (+)
- new net +5V: C8.1, U4.8 (V+)
- new net GND: C10.1, C8.2, R17.2, R20.2, U4.4 (V-), U4.5 (+)

Commit message: aaa
Parts:
- removed D4: D, symbol Device:D
- added D2, D5: D_Schottky, Diode_SMD:D_SOD-123, symbol Device:D_Schottky
- added JP1: Jumper_3_Bridged12, Jumper:SolderJumper-3_P1.3mm_Bridged12_RoundedPad1.0x1.5mm_NumberLabels, symbol Jumper:Jumper_3_Bridged12
- added R21: 10k, Resistor_SMD:R_0805_2012Metric, symbol Device:R
- added RV2, RV3, RV4: 10k, symbol Device:R_Potentiometer
- added U2: LM393, Package_SO:SOIC-8_3.9x4.9mm_P1.27mm, symbol Comparator:LM393
Connections:
- net +3V3: now also R21.1
- net +5V: now also RV2.3
- net GND: now also D2.2 (A), RV2.1
- net at R15.2, R16.1, U4.2 (-): now also RV4.1
- net at C9.2, R17.1, R18.2: now also D2.1 (K), RV3.2
- net at R18.1, R19.2, U4.6 (-): now also RV3.1
- net at U4.7: now also D5.2 (A)
- net at C10.2, R19.1, R20.1: now also D5.1 (K), U2.5 (+)
- net RAD_in: now reaches R16.2
- net RAD_in: now also RV4.2
- new net: JP1.2 (C), U2.6 (-)
- new net: JP1.3 (B), RV2.2
- new net 0.5V: JP1.1 (A)
- new net RAD_out: R21.2, U2.7
- no-connect marks 0 -> 2
Other:
- moved on the sheet: C10, C8, C9, R15, R16, R17, R18, R19, R20, U4A, U4B, U4C

Commit message: aaa
Parts:
- RV2, RV3, RV4: footprint (none) -> Potentiometer_SMD:Potentiometer_Bourns_TC33X_Vertical
Changed lines of the file:
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@@
 			)
 		)
-		(property "Footprint" ""
+		(property "Footprint" "Potentiometer_SMD:Potentiometer_Bourns_TC33X_Vertical"
 			(at 209.55 107.95 0)
 			(effects
@@
 			)
 		)
-		(property "Footprint" ""
+		(property "Footprint" "Potentiometer_SMD:Potentiometer_Bourns_TC33X_Vertical"
 			(at 50.8 101.6 0)
 			(effects
@@
 			)
 		)
-		(property "Footprint" ""
+		(property "Footprint" "Potentiometer_SMD:Potentiometer_Bourns_TC33X_Vertical"
 			(at 133.35 88.9 0)
 			(effects

Commit message: aaa
Parts:
- C8: value 100n -> 100n
- U4: footprint (none) -> Package_SO:SOIC-8_3.9x4.9mm_P1.27mm
- renumbered D2 to D3, D5 to D4, JP1 to JP2, R16 to R15, R15 to R16, RV4 to RV3, RV3 to RV4, RV2 to RV5, U2 to U3
Connections:
- net at R15.1, R16.2, U4.2 (-): now also RV3.3; no longer RV3.1
Other:
- moved on the sheet: RV3
