File: FYP-METRO-SHIELD.kicad_sch (KiCad schematic)
At the start: 4 parts, among them J1 Power, J2 Digital/PWM, J3 Analog, J4 Digital/PWM

Commit message: LOL
Parts:
- added J5: Conn_01x08, Connector_PinSocket_2.54mm:PinSocket_1x08_P2.54mm_Vertical, symbol Connector_Generic:Conn_01x08
Connections:
- net +3V3: now also J5.1 (Pin_1)
- net +5V: now also J5.8 (Pin_8)
- net GND: now also J5.2 (Pin_2), J5.7 (Pin_7)
- net IR Sensor/PT_in: now also J5.4 (Pin_4)
- net Magnet Sensor/MAG_in: now also J5.3 (Pin_3)
- net Ultrasonic Sesnor/US_in: now also J5.5 (Pin_5)

Commit message: aaa
Parts:
- removed J5: Conn_01x08, Connector_PinSocket_2.54mm:PinSocket_1x08_P2.54mm_Vertical, symbol Connector_Generic:Conn_01x08
- added J?: Conn_01x04_Socket, Connector_PinHeader_2.54mm:PinHeader_1x04_P2.54mm_Vertical, symbol Connector:Conn_01x04_Socket
- added J? (x2): Conn_01x02_Socket, Connector_PinHeader_2.54mm:PinHeader_1x02_P2.54mm_Vertical, symbol Connector:Conn_01x02_Socket
- added J?: Screw_Terminal_01x02, symbol Connector:Screw_Terminal_01x02
- added J?: Conn_01x04_Socket, symbol Connector:Conn_01x04_Socket
Connections:
- net +3V3: now also J?.1 (Pin_1), J?.2 (Pin_2)
- net +5V: now also J?.1 (Pin_1), J?.1 (Pin_1)
- net GND: now also J?.1 (Pin_1), J?.1 (Pin_1), J?.3 (Pin_3)
- net IR Sensor/PT_in: now also J?.4 (Pin_4)
- net Magnet Sensor/MAG_in: now also J?.2 (Pin_2)
- net Ultrasonic Sensor/US_in: now also J?.2 (Pin_2)
- net VCC: now also J?.2 (Pin_2)
- new net Radio/RAD_in: J?.2 (Pin_2)
Other:
- sheet Ultrasonic Sesnor renamed Ultrasonic Sensor
- sheet IR Sensor: file SENSRO_IR.kicad_sch -> SENSOR_IR.kicad_sch
- sheet Radio ports: added RAD_in, RAD_out; removed none

Commit message: aaa
Parts:
- removed J?: Screw_Terminal_01x02, symbol Connector:Screw_Terminal_01x02
- removed J?: Conn_01x04_Socket, symbol Connector:Conn_01x04_Socket

Commit message: aaa
Parts:
- gave numbers to parts that had none: 3
Changed lines of the file:
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@@
 		(dnp no)
 		(fields_autoplaced yes)
-		(property "Reference" "J?"
+		(property "Reference" "J7"
 			(at 204.47 71.1199 0)
 			(effects
@@
 			(project ""
 				(path "/e63e39d7-6ac0-4ffd-8aa3-1841a4541b55"
-					(reference "J?")
+					(reference "J7")
 					(unit 1)
 				)
@@
 		(on_board yes)
 		(dnp no)
-		(property "Reference" "#PWR026"
+		(property "Reference" "#PWR09"
 			(at 191.77 73.66 0)
 			(effects
@@
 			(project "FYP-METRO-SHIELD"
 				(path "/e63e39d7-6ac0-4ffd-8aa3-1841a4541b55"
-					(reference "#PWR026")
+					(reference "#PWR09")
 					(unit 1)
 				)
@@
 		(on_board yes)
 		(dnp no)
-		(property "Reference" "#PWR027"
+		(property "Reference" "#PWR06"
 			(at 97.79 104.14 0)
 			(effects
@@
 			(project "FYP-METRO-SHIELD"
 				(path "/e63e39d7-6ac0-4ffd-8aa3-1841a4541b55"
-					(reference "#PWR027")
+					(reference "#PWR06")
 					(unit 1)
 				)
@@
 		(dnp no)
 		(fields_autoplaced yes)
-		(property "Reference" "J?"
+		(property "Reference" "J5"
 			(at 97.155 99.06 0)
 			(effects
@@
 			(project "FYP-METRO-SHIELD"
 				(path "/e63e39d7-6ac0-4ffd-8aa3-1841a4541b55"
-					(reference "J?")
+					(reference "J5")
 					(unit 1)
 				)
@@
 		(on_board yes)
 		(dnp no)
-		(property "Reference" "#PWR024"
+		(property "Reference" "#PWR08"
 			(at 201.93 68.58 0)
 			(effects
@@
 			(project "FYP-METRO-SHIELD"
 				(path "/e63e39d7-6ac0-4ffd-8aa3-1841a4541b55"
-					(reference "#PWR024")
+					(reference "#PWR08")
 					(unit 1)
 				)
@@
 		(dnp no)
 		(fields_autoplaced yes)
-		(property "Reference" "J?"
+		(property "Reference" "J6"
 			(at 173.355 99.06 0)
 			(effects
@@
 			(project ""
 				(path "/e63e39d7-6ac0-4ffd-8aa3-1841a4541b55"
-					(reference "J?")
+					(reference "J6")
 					(unit 1)
 				)
@@
 		(dnp no)
 		(fields_autoplaced yes)
-		(property "Reference" "#PWR025"
+		(property "Reference" "#PWR07"
 			(at 173.99 104.14 0)
 			(effects
@@
 			(project ""
 				(path "/e63e39d7-6ac0-4ffd-8aa3-1841a4541b55"
-					(reference "#PWR025")
-					(unit 1)
-				)
+					(reference "#PWR07")
+					(unit 1)
+				)

Commit message: Add files via upload
Parts:
- removed J7: Conn_01x04_Socket, Connector_PinHeader_2.54mm:PinHeader_1x04_P2.54mm_Vertical, symbol Connector:Conn_01x04_Socket
- added D5: LED, LED_THT:LED_D3.0mm, symbol Device:LED
- added J10: Conn_01x03_Socket, Connector_PinHeader_2.54mm:PinHeader_1x03_P2.54mm_Vertical, symbol Connector:Conn_01x03_Socket
- added J7: Conn_01x02_Socket, Connector_PinHeader_2.54mm:PinHeader_1x02_P2.54mm_Vertical, symbol Connector:Conn_01x02_Socket
- added R22: 3.3k, Resistor_THT:R_Axial_DIN0204_L3.6mm_D1.6mm_P5.08mm_Horizontal, symbol Device:R
Connections:
- net +5V: now also J10.1 (Pin_1), R22.1
- net GND: now also D5.1 (K), J10.3 (Pin_3), J7.2 (Pin_2)
- net IR Sensor/PT_in: now also J7.1 (Pin_1)
- net Magnet Sensor/MAG_in: now also J10.2 (Pin_2)
- net SCL/A5: no longer J2.1 (Pin_1)
- net SDA/A4: no longer J2.2 (Pin_2)
- new net: D5.2 (A), R22.2
- no-connect marks 1 -> 3
