File: SENSOR_IR.kicad_sch (KiCad schematic)
At the start: 7 parts, among them Q1 BC847

Commit message: aaa
Parts:
- added JP?: Jumper_3_Bridged12, Jumper:SolderJumper-3_P1.3mm_Bridged12_RoundedPad1.0x1.5mm_NumberLabels, symbol Jumper:Jumper_3_Bridged12
- added RV?: 10k, symbol Device:R_Potentiometer
Connections:
- net +3V3: now also JP?.1 (A); no longer R1.1, R2.1, R3.1
- net at C2.1, Q1.3 (C), R3.2: now also RV?.1
- new net: JP?.2 (C), R1.1, R2.1, R3.1, RV?.2
- new net +5V: JP?.3 (B)
- no-connect marks 0 -> 1
Other:
- moved on the sheet: C2, R4

Commit message: aaa
Parts:
- RV?: footprint (none) -> Potentiometer_SMD:Potentiometer_Bourns_TC33X_Vertical
Changed lines of the file:
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@@
 			)
 		)
-		(property "Footprint" ""
+		(property "Footprint" "Potentiometer_SMD:Potentiometer_Bourns_TC33X_Vertical"
 			(at 165.1 95.25 0)
 			(effects

Commit message: aaa
Parts:
- gave numbers to parts that had none: 2
Connections:
- net at C2.1, Q1.3 (C), R3.2: now also RV1.3; no longer RV1.1
Other:
- moved on the sheet: RV1
Changed lines of the file:
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@@
 		(dnp no)
 		(fields_autoplaced yes)
-		(property "Reference" "#PWR07"
+		(property "Reference" "#PWR010"
 			(at 111.76 88.9 0)
 			(effects
@@
 			(project ""
 				(path "/e63e39d7-6ac0-4ffd-8aa3-1841a4541b55/0396caee-4752-41d0-833d-b755c6ba6b29"
-					(reference "#PWR07")
+					(reference "#PWR010")
 					(unit 1)
 				)
@@
 	(symbol
 		(lib_id "Device:R_Potentiometer")
-		(at 165.1 95.25 180)
-		(unit 1)
-		(exclude_from_sim no)
-		(in_bom yes)
-		(on_board yes)
-		(dnp no)
-		(fields_autoplaced yes)
-		(property "Reference" "RV?"
+		(at 165.1 95.25 0)
+		(mirror y)
+		(unit 1)
+		(exclude_from_sim no)
+		(in_bom yes)
+		(on_board yes)
+		(dnp no)
+		(property "Reference" "RV1"
 			(at 171.45 95.25 90)
 			(effects
@@
 			(project "FYP-METRO-SHIELD"
 				(path "/e63e39d7-6ac0-4ffd-8aa3-1841a4541b55/0396caee-4752-41d0-833d-b755c6ba6b29"
-					(reference "RV?")
+					(reference "RV1")
 					(unit 1)
 				)
@@
 		(dnp no)
 		(fields_autoplaced yes)
-		(property "Reference" "#PWR041"
+		(property "Reference" "#PWR011"
 			(at 116.84 88.9 0)
 			(effects
@@
 			(project ""
 				(path "/e63e39d7-6ac0-4ffd-8aa3-1841a4541b55/0396caee-4752-41d0-833d-b755c6ba6b29"
-					(reference "#PWR041")
+					(reference "#PWR011")
 					(unit 1)
 				)
@@
 		(dnp no)
 		(fields_autoplaced yes)
-		(property "Reference" "#PWR010"
+		(property "Reference" "#PWR013"
 			(at 190.5 127 0)
 			(effects
@@
 			(project "FYP-METRO-SHIELD"
 				(path "/e63e39d7-6ac0-4ffd-8aa3-1841a4541b55/0396caee-4752-41d0-833d-b755c6ba6b29"
-					(reference "#PWR010")
+					(reference "#PWR013")
 					(unit 1)
 				)
@@
 		(dnp no)
 		(fields_autoplaced yes)
-		(property "Reference" "#PWR09"
+		(property "Reference" "#PWR012"
 			(at 152.4 127 0)
 			(effects
@@
 			(project "FYP-METRO-SHIELD"
 				(path "/e63e39d7-6ac0-4ffd-8aa3-1841a4541b55/0396caee-4752-41d0-833d-b755c6ba6b29"
-					(reference "#PWR09")
+					(reference "#PWR012")
 					(unit 1)
 				)
@@
 		(dnp no)
 		(fields_autoplaced yes)
-		(property "Reference" "JP?"
+		(property "Reference" "JP1"
 			(at 114.3 85.09 0)
 			(effects
@@
 			(project "FYP-METRO-SHIELD"
 				(path "/e63e39d7-6ac0-4ffd-8aa3-1841a4541b55/0396caee-4752-41d0-833d-b755c6ba6b29"
-					(reference "JP?")
-					(unit 1)
-				)
+					(reference "JP1")
+					(unit 1)
+				)

Commit message: Add files via upload
Parts:
- removed JP1: Jumper_3_Bridged12, Jumper:SolderJumper-3_P1.3mm_Bridged12_RoundedPad1.0x1.5mm_NumberLabels, symbol Jumper:Jumper_3_Bridged12
- removed Q1: BC847, Package_TO_SOT_SMD:SOT-23, symbol Transistor_BJT:BC847
- removed RV1: 10k, Potentiometer_SMD:Potentiometer_Bourns_TC33X_Vertical, symbol Device:R_Potentiometer
- added J8: Conn_01x03_Pin, Connector_PinHeader_2.54mm:PinHeader_1x03_P2.54mm_Vertical, symbol Connector:Conn_01x03_Pin
- added Q1: BC547, Package_TO_SOT_THT:TO-92_Inline, symbol Transistor_BJT:BC547
- C1, C2: value 0.1u -> 100n; footprint Capacitor_SMD:C_0805_2012Metric -> Capacitor_THT:C_Disc_D3.0mm_W2.0mm_P2.50mm
- R1, R3, R4: footprint Resistor_SMD:R_0805_2012Metric -> Resistor_THT:R_Axial_DIN0204_L3.6mm_D1.6mm_P5.08mm_Horizontal
- R2: value 370k -> 390k; footprint Resistor_SMD:R_0805_2012Metric -> Resistor_THT:R_Axial_DIN0204_L3.6mm_D1.6mm_P5.08mm_Horizontal
Connections:
- net +3V3: now also J8.3 (Pin_3)
- net +5V: now also J8.1 (Pin_1)
- net GND: now also Q1.3 (E)
- net at R1.1, R2.1, R3.1: now also J8.2 (Pin_2)
- net at C2.1, R3.2: now also Q1.1 (C)
- net at C1.2, R2.2: now also Q1.2 (B)
- no-connect marks 1 -> 0
